Commit message: Updated the meshes and urdf

File: src/bot_description/urdf/bot.xacro (robot description, xacro)
@@ -13,18 +13,19 @@
     <origin xyz="0.0 0.0 0.010" rpy="0 0 0"/>
   </joint>
-  <link name="base_link">
-    <inertial>
-      <origin
-        xyz="-0.027396 1.3878E-17 -0.0041809"
-        rpy="0 0 0" />
-      <mass
-        value="0.11165" />
-      <inertia
-        ixx="0.00017984"
-        ixy="-9.8938E-20"
-        ixz="-5.4132E-21"
-        iyy="0.00051834"
-        iyz="4.6587E-21"
-        izz="0.00068061" />
+  <link
+    name="base_link">
+    <inertial>
+      <origin
+        xyz="-0.038188 -2.7756E-17 0"
+        rpy="0 0 0" />
+      <mass
+        value="0.08" />
+      <inertia
+        ixx="0.0001804"
+        ixy="-9.7007E-20"
+        ixz="-3.3783E-22"
+        iyy="0.00053906"
+        iyz="-8.3789E-23"
+        izz="0.0007194" />
     </inertial>
     <visual>
@@ -39,5 +40,5 @@
         name="">
         <color
-          rgba="0.79216 0.81961 0.93333 1" />
+          rgba="1 1 1 0.32" />
       </material>
     </visual>
@@ -53,45 +54,363 @@
   </link>
   <link
-    name="caster">
-    <inertial>
-      <origin
-        xyz="2.398E-09 -5.9697E-09 -0.02447"
-        rpy="0 0 0" />
-      <mass
-        value="0.074554" />
-      <inertia
-        ixx="2.263E-05"
-        ixy="-5.1952E-13"
-        ixz="2.1696E-13"
-        iyy="2.263E-05"
-        iyz="-8.3514E-13"
-        izz="2.7097E-05" />
-    </inertial>
-    <visual>
-      <origin
-        xyz="0 0 0"
-        rpy="0 0 0" />
-      <geometry>
-        <mesh
-          filename="package://bot_description/meshes/caster.STL" />
-      </geometry>
-      <material
-        name="">
-        <color
-          rgba="0.79216 0.81961 0.93333 1" />
-      </material>
-    </visual>
-    <collision>
-      <origin
-        xyz="0 0 0"
-        rpy="0 0 0" />
-      <geometry>
-        <mesh
-          filename="package://bot_description/meshes/caster.STL" />
-      </geometry>
-    </collision>
-  </link>
-  <joint
-    name="caster_joint"
+    name="right_bracket">
+    <inertial>
+      <origin
+        xyz="-0.010316 0.013793 -3.4694E-18"
+        rpy="0 0 0" />
+      <mass
+        value="0.045578" />
+      <inertia
+        ixx="2.1019E-05"
+        ixy="3.1847E-06"
+        ixz="-3.4097E-21"
+        iyy="1.1949E-05"
+        iyz="7.5589E-23"
+        izz="1.6242E-05" />
+    </inertial>
+    <visual>
+      <origin
+        xyz="0 0 0"
+        rpy="0 0 0" />
+      <geometry>
+        <mesh
+          filename="package://bot_description/meshes/right_bracket.STL" />
+      </geometry>
+      <material
+        name="">
+        <color
+          rgba="0.52941 0.54902 0.54902 1" />
+      </material>
+    </visual>
+    <collision>
+      <origin
+        xyz="0 0 0"
+        rpy="0 0 0" />
+      <geometry>
+        <mesh
+          filename="package://bot_description/meshes/right_bracket.STL" />
+      </geometry>
+    </collision>
+  </link>
+  <joint
+    name="right_bracket_joint"
+    type="fixed">
+    <origin
+      xyz="0 -0.0475 -0.001"
+      rpy="-1.5708 0 1.5708" />
+    <parent
+      link="base_link" />
+    <child
+      link="right_bracket" />
+    <axis
+      xyz="0 0 0" />
+  </joint>
+  <link
+    name="right_coupler">
+    <inertial>
+      <origin
+        xyz="-8.1082E-06 -0.015391 1.4045E-05"
+        rpy="0 0 0" />
+      <mass
+        value="0.024489" />
+      <inertia
+        ixx="2.132E-06"
+        ixy="2.5519E-09"
+        ixz="-7.5949E-10"
+        iyy="5.3128E-07"
+        iyz="-4.42E-09"
+        izz="2.1328E-06" />
+    </inertial>
+    <visual>
+      <origin
+        xyz="0 0 0"
+        rpy="0 0 0" />
+      <geometry>
+        <mesh
+          filename="package://bot_description/meshes/right_coupler.STL" />
+      </geometry>
+      <material
+        name="">
+        <color
+          rgba="0.64706 0.51765 0 1" />
+      </material>
+    </visual>
+    <collision>
+      <origin
+        xyz="0 0 0"
+        rpy="0 0 0" />
+      <geometry>
+        <mesh
+          filename="package://bot_description/meshes/right_coupler.STL" />
+      </geometry>
+    </collision>
+  </link>
+  <joint
+    name="right_coupler_joint"
+    type="fixed">
+    <origin
+      xyz="-0.036008 0.0304 0"
+      rpy="-3.1416 0.97109 1.5708" />
+    <parent
+      link="right_bracket" />
+    <child
+      link="right_coupler" />
+    <axis
+      xyz="0 1 0" />
+  </joint>
+  <link
+    name="right_wheel">
+    <inertial>
+      <origin
+        xyz="-6.1785E-11 -1.3014E-11 0.014376"
+        rpy="0 0 0" />
+      <mass
+        value="0.3445" />
+      <inertia
+        ixx="0.00022322"
+        ixy="-1.5874E-13"
+        ixz="-3.4623E-13"
+        iyy="0.00022322"
+        iyz="-1.3247E-14"
+        izz="0.00035265" />
+    </inertial>
+    <visual>
+      <origin
+        xyz="0 0 0"
+        rpy="0 0 0" />
+      <geometry>
+        <mesh
+          filename="package://bot_description/meshes/right_wheel.STL" />
+      </geometry>
+      <material
+        name="">
+        <color
+          rgba="0.29804 0.29804 0.29804 1" />
+      </material>
+    </visual>
+    <collision>
+      <origin
+        xyz="0 0 0"
+        rpy="0 0 0" />
+      <geometry>
+        <mesh
+          filename="package://bot_description/meshes/right_wheel.STL" />
+      </geometry>
+    </collision>
+  </link>
+  <joint
+    name="right_wheel_joint"
+    type="continuous">
+    <origin
+      xyz="0 0 0"
+      rpy="-1.5708 0.5236 -3.1416" />
+    <parent
+      link="right_coupler" />
+    <child
+      link="right_wheel" />
+    <axis
+      xyz="0 0 1" />
+  </joint>
+  <link
+    name="left_bracket">
+    <inertial>
+      <origin
+        xyz="-0.010316 0.013793 -1.2143E-17"
+        rpy="0 0 0" />
+      <mass
+        value="0.045578" />
+      <inertia
+        ixx="2.1019E-05"
+        ixy="3.1847E-06"
+        ixz="3.2297E-21"
+        iyy="1.1949E-05"
+        iyz="1.7687E-20"
+        izz="1.6242E-05" />
+    </inertial>
+    <visual>
+      <origin
+        xyz="0 0 0"
+        rpy="0 0 0" />
+      <geometry>
+        <mesh
+          filename="package://bot_description/meshes/left_bracket.STL" />
+      </geometry>
+      <material
+        name="">
+        <color
+          rgba="0.52941 0.54902 0.54902 1" />
+      </material>
+    </visual>
+    <collision>
+      <origin
+        xyz="0 0 0"
+        rpy="0 0 0" />
+      <geometry>
+        <mesh
+          filename="package://bot_description/meshes/left_bracket.STL" />
+      </geometry>
+    </collision>
+  </link>
+  <joint
+    name="left_bracket_joint"
+    type="fixed">
+    <origin
+      xyz="0 0.0475 -0.001"
+      rpy="-1.5708 0 -1.5708" />
+    <parent
+      link="base_link" />
+    <child
+      link="left_bracket" />
+    <axis
+      xyz="0 0 0" />
+  </joint>
+  <link
+    name="left_coupler">
+    <inertial>
+      <origin
+        xyz="-8.0592E-06 -0.015391 1.4073E-05"
+        rpy="0 0 0" />
+      <mass
+        value="0.024489" />
+      <inertia
+        ixx="2.132E-06"
+        ixy="2.5519E-09"
+        ixz="-7.5949E-10"
+        iyy="5.3128E-07"
+        iyz="-4.42E-09"
+        izz="2.1328E-06" />
+    </inertial>
+    <visual>
+      <origin
+        xyz="0 0 0"
+        rpy="0 0 0" />
+      <geometry>
+        <mesh
+          filename="package://bot_description/meshes/left_coupler.STL" />
+      </geometry>
+      <material
+        name="">
+        <color
+          rgba="0.64706 0.51765 0 1" />
+      </material>
+    </visual>
+    <collision>
+      <origin
+        xyz="0 0 0"
+        rpy="0 0 0" />
+      <geometry>
+        <mesh
+          filename="package://bot_description/meshes/left_coupler.STL" />
+      </geometry>
+    </collision>
+  </link>
+  <joint
+    name="left_coupler_joint"
+    type="fixed">
+    <origin
+      xyz="-0.036008 0.0304 0"
+      rpy="-3.1416 1.1233 1.5708" />
+    <parent
+      link="left_bracket" />
+    <child
+      link="left_coupler" />
+    <axis
+      xyz="0 1 0" />
+  </joint>
+  <link
+    name="left_wheel">
+    <inertial>
+      <origin
+        xyz="-5.6627E-08 -1.2522E-11 0.014376"
+        rpy="0 0 0" />
+      <mass
+        value="0.3445" />
+      <inertia
+        ixx="0.00022322"
+        ixy="-1.5874E-13"
+        ixz="-3.4751E-13"
+        iyy="0.00022322"
+        iyz="-1.2402E-14"
+        izz="0.00035265" />
+    </inertial>
+    <visual>
+      <origin
+        xyz="0 0 0"
+        rpy="0 0 0" />
+      <geometry>
+        <mesh
+          filename="package://bot_description/meshes/left_wheel.STL" />
+      </geometry>
+      <material
+        name="">
+        <color
+          rgba="0.29804 0.29804 0.29804 1" />
+      </material>
+    </visual>
+    <collision>
+      <origin
+        xyz="0 0 0"
+        rpy="0 0 0" />
+      <geometry>
+        <mesh
+          filename="package://bot_description/meshes/left_wheel.STL" />
+      </geometry>
+    </collision>
+  </link>
+  <joint
+    name="left_wheel_joint"
+    type="continuous">
+    <origin
+      xyz="0 0 0"
+      rpy="-1.5708 0.5236 -3.1416" />
+    <parent
+      link="left_coupler" />
+    <child
+      link="left_wheel" />
+    <axis
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
File: src/bot_description/urdf/gazebo_plugins.xacro (robot description, xacro)
@@ -15,10 +15,10 @@
       <legacyMode>false</legacyMode>
       <updateRate>30</updateRate>
-      <leftJoint>left_joint</leftJoint>
-      <rightJoint>right_joint</rightJoint>
-      <wheelSeparation>0.160</wheelSeparation>
-      <wheelDiameter>0.066</wheelDiameter>
-      <wheelAcceleration>1</wheelAcceleration>
-      <wheelTorque>10</wheelTorque>
+      <leftJoint>left_wheel_joint</leftJoint>
+      <rightJoint>right_wheel_joint</rightJoint>
+      <wheelSeparation>0.25</wheelSeparation>
+      <wheelDiameter>0.040</wheelDiameter>
+      <wheelAcceleration>2</wheelAcceleration>
+      <wheelTorque>50</wheelTorque>
       <rosDebugLevel>na</rosDebugLevel>
     </plugin>

File: src/bot_description/urdf/gazebo_properties.xacro (robot description, xacro)
@@ -5,11 +5,23 @@
     <material>Gazebo/White</material>
   </gazebo>
+  <gazebo reference="right_bracket">
+    <material>Gazebo/FlatBlack</material>
+  </gazebo>
+  <gazebo reference="left_bracket">
+    <material>Gazebo/FlatBlack</material>
+  </gazebo>
+  <gazebo reference="right_coupler">
+    <material>Gazebo/Yellow</material>
+  </gazebo>
+  <gazebo reference="left_coupler">
+    <material>Gazebo/Yellow</material>
+  </gazebo>
   <gazebo reference="left_wheel">
     <mu1>0.1</mu1>
     <mu2>0.1</mu2>
-    <kp>500000.0</kp>
-    <kd>10.0</kd>
+    <kp>1000000.0</kp>
+    <kd>100.0</kd>
     <minDepth>0.001</minDepth>
-    <maxVel>0.1</maxVel>
+    <maxVel>10.0</maxVel>
     <fdir1>1 0 0</fdir1>
     <material>Gazebo/FlatBlack</material>
@@ -18,12 +30,15 @@
     <mu1>0.1</mu1>
     <mu2>0.1</mu2>
-    <kp>500000.0</kp>
-    <kd>10.0</kd>
+    <kp>1000000.0</kp>
+    <kd>100.0</kd>
     <minDepth>0.001</minDepth>
-    <maxVel>0.1</maxVel>
+    <maxVel>10.0</maxVel>
     <fdir1>1 0 0</fdir1>
     <material>Gazebo/FlatBlack</material>
   </gazebo>
-  <gazebo reference="caster">
+  <gazebo reference="caster_one">
+    <material>Gazebo/Red</material>
+  </gazebo>
+  <gazebo reference="caster_two">
     <mu1>0.1</mu1>
     <mu2>0.1</mu2>
@@ -31,11 +46,41 @@
     <kd>100.0</kd>
     <minDepth>0.001</minDepth>
-    <maxVel>1.0</maxVel>
+    <maxVel>10.0</maxVel>
+    <material>Gazebo/White</material>
+  </gazebo>
+  <gazebo reference="back_standoff_one">
+    <material>Gazebo/Yellow</material>
+  </gazebo>
+  <gazebo reference="back_standoff_two">
+    <material>Gazebo/Yellow</material>
+  </gazebo>
+  <gazebo reference="back_standoff_three">
+    <material>Gazebo/Yellow</material>
+  </gazebo>
+  <gazebo reference="back_standoff_four">
+    <material>Gazebo/Yellow</material>
+  </gazebo>
+  <gazebo reference="front_standoff_one">
+    <material>Gazebo/Yellow</material>
+  </gazebo>
+  <gazebo reference="front_standoff_two">
+    <material>Gazebo/Yellow</material>
+  </gazebo>
+  <gazebo reference="front_standoff_three">
+    <material>Gazebo/Yellow</material>
+  </gazebo>
+  <gazebo reference="front_standoff_four">
+    <material>Gazebo/Yellow</material>
+  </gazebo>
+  <gazebo reference="back_cover">
+    <material>Gazebo/White</material>
+  </gazebo>
+  <gazebo reference="front_cover">
+    <material>Gazebo/White</material>
+  </gazebo>
+  <gazebo reference="lidar">
     <material>Gazebo/FlatBlack</material>
   </gazebo>
-  <!--gazebo reference="base_scan">
-    <material>Gazebo/FlatBlack</material>
-  </gazebo>
-  <gazebo reference="imu_link">
+  <!--gazebo reference="imu_link">
     <sensor type="imu" name="imu">
       <always_on>true</always_on>
